Commit message: Fixed for simulation

File: simulation/xacro/mylaser.xacro (robot description, xacro)
@@ -28,5 +28,5 @@
 			<origin xyz="0 0 0" rpy="0 0 0"/>
 			<geometry>
-				<mesh filename="file:///home/patri/catkin_ws/src/simulation/meshes/hokuyo.dae"/>
+				<mesh filename="file:///yourpath/catkin_ws/src/simulation/meshes/hokuyo.dae"/>
 			</geometry>
 		</visual>
